Commit message: Fix real-hardware URDF gripper model and sync controller joint config

File: brainswarm_ws/src/roboflex_description/urdf/real_hardware.urdf.xacro (robot description, xacro)
@@ -98,5 +98,5 @@
       xyz="0 0 1" />
     <limit
-      lower="-1.57"
+      lower="0.0"
       upper="1.57"
       effort="1000"
@@ -157,5 +157,5 @@
     <limit
       lower="-1.57"
-      upper="1.57"
+      upper="0.523333"
       effort="1000"
       velocity="1000" />
@@ -215,10 +215,10 @@
     <limit
       lower="-1.57"
-      upper="1.57"
-      effort="1000"
-      velocity="1000" />
-  </joint>
-  <link
-    name="gripper_body_link">
+      upper="-0.174444"
+      effort="1000"
+      velocity="1000" />
+  </joint>
+  <link
+    name="link_4">
     <inertial>
       <origin
@@ -260,5 +260,5 @@
   </link>
   <joint
-    name="joint_gripper_body"
+    name="joint_4"
     type="revolute">
     <origin
@@ -268,18 +268,18 @@
       link="link_3" />
     <child
-      link="gripper_body_link" />
+      link="link_4" />
     <axis
       xyz="0 1 0" />
     <limit
-      lower="-1"
-      upper="1"
-      effort="1000"
-      velocity="1000" />
-  </joint>
-  <link
-    name="gripper_left_link">
-    <inertial>
-      <origin
-        xyz="0.0764884076472838 -0.0289481833034687 0.00870239087002106"
+      lower="-1.57"
+      upper="0.523333"
+      effort="1000"
+      velocity="1000" />
+  </joint>
+  <link
+    name="left_finger_link">
+    <inertial>
+      <origin
+        xyz="0 0 0"
         rpy="0 0 0" />
       <mass
@@ -317,27 +317,62 @@
     </collision>
   </link>
-  <joint
-    name="joint_gripper_left_part"
-    type="prismatic">
+  <link name="gripper_drive_link" />
+  <link name="gripper_actuator_link" />
+  <joint
+    name="joint_gripper_mount"
+    type="fixed">
+    <origin
+      xyz="0.0718 -0.03 0.008"
+      rpy="0 0 0" />
+    <parent
+      link="link_4" />
+    <child
+      link="gripper_drive_link" />
+  </joint>
+  <joint
+    name="joint_gripper"
+    type="revolute">
     <origin
       xyz="0 0 0"
       rpy="0 0 0" />
     <parent
-      link="gripper_body_link" />
-    <child
-      link="gripper_left_link" />
+      link="gripper_drive_link" />
+    <child
+      link="gripper_actuator_link" />
     <axis
       xyz="0 1 0" />
     <limit
-      lower="-0.4"
-      upper="0"
-      effort="1000"
-      velocity="1000" />
-  </joint>
-  <link
-    name="gripper_right_link">
-    <inertial>
-      <origin
-        xyz="0.0764887069201697 -0.0464089888469002 0.00870242590433329"
+      lower="0.0"
+      upper="0.523333"
+      effort="1000"
+      velocity="1000" />
+  </joint>
+  <joint
+    name="joint_gripper_left_finger"
+    type="prismatic">
+    <origin
+      xyz="0 0.001 0"
+      rpy="0 -0.118 0" />
+    <parent
+      link="gripper_drive_link" />
+    <child
+      link="left_finger_link" />
+    <axis
+      xyz="0 1 0" />
+    <limit
+      lower="-0.006"
+      upper="0.0"
+      effort="1000"
+      velocity="1000" />
+    <mimic
+      joint="joint_gripper"
+      multiplier="0.011465"
+      offset="0.0" />
+  </joint>
+  <link
+    name="right_finger_link">
+    <inertial>
+      <origin
+        xyz="0 0 0"
         rpy="0 0 0" />
       <mass
@@ -379,17 +414,21 @@
     type="prismatic">
     <origin
-      xyz="0 0 0"
-      rpy="0 0 0" />
-    <parent
-      link="gripper_body_link" />
-    <child
-      link="gripper_right_link" />
+      xyz="0 -0.001 0"
+      rpy="0 -0.118 0" />
+    <parent
+      link="gripper_drive_link" />
+    <child
+      link="right_finger_link" />
     <axis
       xyz="0 1 0" />
     <limit
-      lower="0"
-      upper="0.4"
-      effort="1000"
-      velocity="1000" />
+      lower="0.0"
+      upper="0.006"
+      effort="1000"
+      velocity="1000" />
+    <mimic
+      joint="joint_gripper"
+      multiplier="-0.011465"
+      offset="0.0" />
   </joint>
   <ros2_control name="RealHardwareSystem" type="system">
@@ -399,5 +438,5 @@
         <joint name="joint_1">
             <command_interface name="position">
-                <param name="min">-1.57</param>
+                <param name="min">0.0</param>
                 <param name="max">1.57</param>
             </command_interface>
@@ -408,6 +447,6 @@
         <joint name="joint_2">
             <command_interface name="position">
-                <param name="min">-2.879793</param>
-                <param name="max">2.879793</param>
+                <param name="min">-1.57</param>
+                <param name="max">0.523333</param>
             </command_interface>
             <state_interface name="position">
@@ -417,6 +456,6 @@
         <joint name="joint_3">
             <command_interface name="position">
-                <param name="min">-2.879793</param>
-                <param name="max">2.879793</param>
+                <param name="min">-1.57</param>
+                <param name="max">-0.174444</param>
             </command_interface>
             <state_interface name="position">
@@ -424,8 +463,8 @@
             </state_interface>
         </joint>
-        <joint name="joint_gripper_body">
+        <joint name="joint_4">
             <command_interface name="position">
-                <param name="min">-2.879793</param>
-                <param name="max">2.879793</param>
+                <param name="min">-1.57</param>
+                <param name="max">0.523333</param>
             </command_interface>
             <state_interface name="position">
@@ -433,8 +472,8 @@
             </state_interface>
         </joint>
-        <joint name="joint_gripper_left_part">
+        <joint name="joint_gripper">
             <command_interface name="position">
                 <param name="min">0</param>
-                <param name="max">1.57</param>
+                <param name="max">0.523333</param>
             </command_interface>
             <state_interface name="position">
